File: blink-twice.kicad_sch (KiCad schematic)
At the start: 13 parts, among them U2 4017, U3 NE555P

Commit message: Groomed, and saved with KiCad 8.
Parts:
- U3: symbol ne555p:NE555P -> local:NE555P
Changed lines of the file:
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@@
+	(wire
+		(pts
+			(xy 209.55 78.74) (xy 209.55 82.55)
+		)
+		(stroke
+			(width 0)
+			(type default)
+		)
+	)
 	(wire
 		(pts
@@
 	)
 	(symbol
-		(lib_id "ne555p:NE555P")
+		(lib_id "local:NE555P")
 		(at 133.35 97.79 0)
 		(unit 1)
@@
 	(symbol
 		(lib_id "power:PWR_FLAG")
-		(at 209.55 82.55 0)
+		(at 209.55 78.74 0)
 		(unit 1)
 		(exclude_from_sim no)
@@
 		(fields_autoplaced yes)
 		(property "Reference" "#FLG01"
-			(at 209.55 80.645 0)
+			(at 209.55 76.835 0)
 			(effects
 				(font
@@
 		)
 		(property "Value" "PWR_FLAG"
-			(at 209.55 78.4169 0)
+			(at 209.55 74.6069 0)
 			(effects
 				(font
@@
 		)
 		(property "Footprint" ""
-			(at 209.55 82.55 0)
+			(at 209.55 78.74 0)
 			(effects
 				(font
@@
 		)
 		(property "Datasheet" "~"
-			(at 209.55 82.55 0)
+			(at 209.55 78.74 0)
 			(effects
 				(font
@@
 		)
 		(property "Description" "Special symbol for telling ERC where power comes from"
-			(at 209.55 82.55 0)
-			(effects
-				(font
+			(at 209.55 78.74 0)
+			(effects
+				(font
